File: pcb/revA/nanit.kicad_pcb (KiCad board)
At the start: 2 copper layers, 31.2 x 53.3 mm, 68 parts, among them J1 USB_B_Micro, J2 Nokia 2660/2760 mini, Q1 BC857, Q2 IRLML6344, Q4 BC847, SW1 Button 1, SW2 Button 2, U1 LTC4054ES5-4.2, U2 ATmega88PA-AU, U3 LT1937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

Commit message: latest pcb and schematics
Parts:
- C13, C14, C15: value 100nF 600V -> 100nF
- C9: value 10pF 1000V (C17UL100J-7ZN-X1T) -> 10pF
- D8: value 18v (BZV55C18) -> BZV55C18
- TP4: value PROG_RST -> RST
