File: pcb/revA/nanit.sch (KiCad schematic (older format))
At the start: 68 parts, among them J1 USB_B_Micro, J2 Nokia 2660/2760 mini, Q1 BC857, Q2 IRLML6344, Q4 BC847, SW1 Button 1, SW2 Button 2, U1 LTC4054ES5-4.2, U2 ATmega88PA-AU, U3 LT1937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

Commit message: latest pcb and schematics
Parts:
- S1: symbol doz:SBM-21 -> nanit-rescue:SBM-21-doz
- TR1: symbol doz:CEEH54 -> nanit-rescue:CEEH54-doz
- U3: symbol doz:LT1937 -> nanit-rescue:LT1937-doz
Changed lines of the file:
@@
 $EndComp
 $Comp
-L doz:SBM-21 S1
+L nanit-rescue:SBM-21-doz S1
 U 1 1 5E383BDC
 P 1200 5200
@@
 Connection ~ 7900 2900
 $Comp
-L doz:CEEH54 TR1
+L nanit-rescue:CEEH54-doz TR1
 U 1 1 5E659661
 P 5300 5050
@@
 	1200 1600 1450 1600
 $Comp
-L doz:LT1937 U3
+L nanit-rescue:LT1937-doz U3
 U 1 1 5E42EB7A
 P 3750 1750
