File: pcb/revD/nanit.kicad_pcb (KiCad board)
At the start: 2 copper layers, 31.2 x 53.3 mm, 71 parts, among them J1 USB_B_Micro, Q1 BC857, Q2 IRLML6344, Q4 BC847, SW1 Button 1, SW2 Button 2, U1 LTC4054ES5-4.2, U2 ATmega328P, U3 CH340G, U4 HT16K33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

Commit message: revD fixes - missing AREF capacitor C7
Parts:
- added C7: 100nF, Capacitor_SMD:C_0805_2012Metric_Pad1.18x1.45mm_HandSolder, B.Cu at (135.3, 117.7)
Connections:
- J1 pad 4: (no net) -> unconnected-(J1-Pad4)
- U2 pad 10: (no net) -> unconnected-(U2-Pad10)
- U2 pad 11: (no net) -> unconnected-(U2-Pad11)
- U2 pad 13: (no net) -> unconnected-(U2-Pad13)
- U2 pad 14: (no net) -> unconnected-(U2-Pad14)
- U2 pad 19: (no net) -> unconnected-(U2-Pad19)
- U2 pad 20: (no net) -> Net-(U2-Pad20)
- U2 pad 22: (no net) -> unconnected-(U2-Pad22)
- U2 pad 23: (no net) -> unconnected-(U2-Pad23)
- U2 pad 24: (no net) -> unconnected-(U2-Pad24)
- U3 pad 10: (no net) -> unconnected-(U3-Pad10)
- U3 pad 11: (no net) -> unconnected-(U3-Pad11)
- U3 pad 12: (no net) -> unconnected-(U3-Pad12)
- U3 pad 14: (no net) -> unconnected-(U3-Pad14)
- U3 pad 15: (no net) -> unconnected-(U3-Pad15)
- U3 pad 9: (no net) -> unconnected-(U3-Pad9)
- U4 pad 10: (no net) -> unconnected-(U4-Pad10)
- U4 pad 11: (no net) -> unconnected-(U4-Pad11)
- U4 pad 12: (no net) -> unconnected-(U4-Pad12)
- U4 pad 13: (no net) -> unconnected-(U4-Pad13)
- U4 pad 14: (no net) -> unconnected-(U4-Pad14)
- U4 pad 15: (no net) -> unconnected-(U4-Pad15)
- U4 pad 16: (no net) -> unconnected-(U4-Pad16)
- U4 pad 17: (no net) -> unconnected-(U4-Pad17)
- U4 pad 7: (no net) -> unconnected-(U4-Pad7)
- U4 pad 8: (no net) -> unconnected-(U4-Pad8)
- U4 pad 9: (no net) -> unconnected-(U4-Pad9)
Routing:
- net Net-(U2-Pad20): track 0.00 -> 2.41 mm, vias 0 -> 1
